File: page11.sch (KiCad schematic (older format))
At the start: 5 parts

Commit message: Schematic update
Connections:
- net GND: now reaches U?.A11 (VSS1)
- net GND: now also U?.A15 (VSS2), U?.A19 (VSS3), U?.A23 (VSS4), U?.A27 (VSS5), U?.A31 (VSS6), U?.A35 (VSS7), U?.A39 (VSS8), U?.A43 (VSS9), U?.A47 (VSS10), U?.AA1 (VSS11), U?.AA16 (VSS12), U?.AA19 (VSS13)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
