File: page3.sch (KiCad schematic (older format))
At the start: 1 part

Commit message: Schematic update.
Parts:
- added R?: 2.2K, symbol Device:R_Small_US
- added R? (x2): 0, symbol Device:R_Small_US
- added R?: 357, symbol Device:R_Small_US
- added R? (x3): 150, symbol Device:R_Small_US
Connections:
- net at U?.AH2 (RESERVED_VSS3): now also R?.2
- net at U?.AH3 (RESERVED_VSS2): now also R?.2
- net at U?.AW1 (VGA_IREF): now also R?.2
- net GND: now reaches U?.AY3 (VGA_IRTN)
- net GND: now also U?.G30 (DDI1_DDCCLK), U?.K30 (DDI1_HPD), R?.1, R?.1, R?.1, R?.1, R?.1, R?.1, R?.1
- net at U?.BC1 (VGA_DDCCLK): now also R?.2
- net at U?.BC2 (VGA_DDCDATA): now also R?.2
- net at U?.P14 (RESERVED_P14): now also R?.2
- net at U?.P30 (DDI1_DDCDATA): now also R?.2
Changed lines of the file:
@@
 	1    0    0    -1
 $EndComp
+$Comp
+L power:GND #PWR?
+U 1 1 5FED669B
+P 10200 2950
+F 0 "#PWR?" H 10200 2700 50  0001 C CNN
+F 1 "GND" V 10205 2822 50  0000 R CNN
+F 2 "" H 10200 2950 50  0001 C CNN
+F 3 "" H 10200 2950 50  0001 C CNN
+	1    10200 2950
+	0    -1   -1   0
+$EndComp
+Wire Wire Line
+	10200 2950 9150 2950
+$Comp
+L power:GND #PWR?
+U 1 1 5FEDAD87
+P 10200 3200
+F 0 "#PWR?" H 10200 2950 50  0001 C CNN
+F 1 "GND" V 10205 3072 50  0000 R CNN
+F 2 "" H 10200 3200 50  0001 C CNN
+F 3 "" H 10200 3200 50  0001 C CNN
+	1    10200 3200
+	0    -1   -1   0
+$EndComp
+Wire Wire Line
+	10200 3200 9150 3200
+$Comp
+L Device:R_Small_US R?
+U 1 1 5FEDC56A
+P 10700 3100
+F 0 "R?" V 10495 3100 50  0000 C CNN
+F 1 "2.2K" V 10586 3100 50  0000 C CNN
+F 2 "" H 10700 3100 50  0001 C CNN
+F 3 "~" H 10700 3100 50  0001 C CNN
+	1    10700 3100
+	0    1    1    0
+$EndComp
+Wire Wire Line
+	9150 3100 10600 3100
+$Comp
+L power:GND #PWR?
+U 1 1 5FEE32CE
+P 11050 3100
+F 0 "#PWR?" H 11050 2850 50  0001 C CNN
+F 1 "GND" V 11055 2972 50  0000 R CNN
+F 2 "" H 11050 3100 50  0001 C CNN
+F 3 "" H 11050 3100 50  0001 C CNN
+	1    11050 3100
+	0    -1   -1   0
+$EndComp
+Wire Wire Line
+	11050 3100 10800 3100
+$Comp
+L Device:R_Small_US R?
+U 1 1 5FEE811A
+P 11000 4200
+F 0 "R?" V 10795 4200 50  0000 C CNN
+F 1 "0" V 10886 4200 50  0000 C CNN
+F 2 "" H 11000 4200 50  0001 C CNN
+F 3 "~" H 11000 4200 50  0001 C CNN
+	1    11000 4200
+	0    1    1    0
+$EndComp
+$Comp
+L Device:R_Small_US R?
+U 1 1 5FEE96DF
+P 10700 4100
+F 0 "R?" V 10495 4100 50  0000 C CNN
+F 1 "0" V 10586 4100 50  0000 C CNN
+F 2 "" H 10700 4100 50  0001 C CNN
+F 3 "~" H 10700 4100 50  0001 C CNN
+	1    10700 4100
+	0    1    1    0
+$EndComp
+Wire Wire Line
+	10600 4100 9150 4100
+Wire Wire Line
+	9150 4200 10900 4200
+$Comp
+L power:GND #PWR?
+U 1 1 5FEFE8F3
+P 11250 4200
+F 0 "#PWR?" H 11250 3950 50  0001 C CNN
+F 1 "GND" V 11255 4072 50  0000 R CNN
+F 2 "" H 11250 4200 50  0001 C CNN
+F 3 "" H 11250 4200 50  0001 C CNN
+	1    11250 4200
+	0    -1   -1   0
+$EndComp
+$Comp
+L power:GND #PWR?
+U 1 1 5FF005E8
+P 11250 4100
+F 0 "#PWR?" H 11250 3850 50  0001 C CNN
+F 1 "GND" V 11255 3972 50  0000 R CNN
+F 2 "" H 11250 4100 50  0001 C CNN
+F 3 "" H 11250 4100 50  0001 C CNN
+	1    11250 4100
+	0    -1   -1   0
+$EndComp
+Wire Wire Line
+	11250 4100 10800 4100
+Wire Wire Line
+	11100 4200 11250 4200
+$Comp
+L Device:R_Small_US R?
+U 1 1 5FF05D8D
+P 10700 4650
+F 0 "R?" V 10495 4650 50  0000 C CNN
+F 1 "357" V 10586 4650 50  0000 C CNN
+F 2 "" H 10700 4650 50  0001 C CNN
+F 3 "~" H 10700 4650 50  0001 C CNN
+	1    10700 4650
+	0    1    1    0
+$EndComp
+Wire Wire Line
+	10600 4650 9150 4650
+$Comp
+L power:GND #PWR?
+U 1 1 5FF05D94
+P 11250 4650
+F 0 "#PWR?" H 11250 4400 50  0001 C CNN
+F 1 "GND" V 11255 4522 50  0000 R CNN
+F 2 "" H 11250 4650 50  0001 C CNN
+F 3 "" H 11250 4650 50  0001 C CNN
+	1    11250 4650
+	0    -1   -1   0
+$EndComp
+Wire Wire Line
+	11250 4650 10800 4650
+$Comp
+L power:GND #PWR?
+U 1 1 5FF093F6
+P 10200 4750
+F 0 "#PWR?" H 10200 4500 50  0001 C CNN
+F 1 "GND" V 10205 4622 50  0000 R CNN
+F 2 "" H 10200 4750 50  0001 C CNN
+F 3 "" H 10200 4750 50  0001 C CNN
+	1    10200 4750
+	0    -1   -1   0
+$EndComp
+Wire Wire Line
+	10200 4750 9150 4750
+$Comp
+L Device:R_Small_US R?
+U 1 1 5FF0E733
+P 11000 5250
+F 0 "R?" V 10795 5250 50  0000 C CNN
+F 1 "150" V 10886 5250 50  0000 C CNN
+F 2 "" H 11000 5250 50  0001 C CNN
+F 3 "~" H 11000 5250 50  0001 C CNN
+	1    11000 5250
+	0    1    1    0
+$EndComp
+$Comp
+L Device:R_Small_US R?
+U 1 1 5FF0E739
+P 10700 5150
+F 0 "R?" V 10495 5150 50  0000 C CNN
+F 1 "150" V 10586 5150 50  0000 C CNN
+F 2 "" H 10700 5150 50  0001 C CNN
+F 3 "~" H 10700 5150 50  0001 C CNN
+	1    10700 5150
+	0    1    1    0
+$EndComp
+Wire Wire Line
+	10600 5150 9150 5150
+Wire Wire Line
+	9150 5250 10900 5250
+$Comp
+L power:GND #PWR?
+U 1 1 5FF0E741
+P 11250 5250
+F 0 "#PWR?" H 11250 5000 50  0001 C CNN
+F 1 "GND" V 11255 5122 50  0000 R CNN
+F 2 "" H 11250 5250 50  0001 C CNN
+F 3 "" H 11250 5250 50  0001 C CNN
+	1    11250 5250
+	0    -1   -1   0
+$EndComp
+$Comp
+L power:GND #PWR?
+U 1 1 5FF0E747
+P 11250 5150
+F 0 "#PWR?" H 11250 4900 50  0001 C CNN
+F 1 "GND" V 11255 5022 50  0000 R CNN
+F 2 "" H 11250 5150 50  0001 C CNN
+F 3 "" H 11250 5150 50  0001 C CNN
+	1    11250 5150
+	0    -1   -1   0
+$EndComp
+Wire Wire Line
+	11250 5150 10800 5150
+Wire Wire Line
+	11100 5250 11250 5250
+$Comp
+L Device:R_Small_US R?
+U 1 1 5FF12FB1
+P 10700 7000
+F 0 "R?" V 10495 7000 50  0000 C CNN
+F 1 "150" V 10586 7000 50  0000 C CNN
+F 2 "" H 10700 7000 50  0001 C CNN
+F 3 "~" H 10700 7000 50  0001 C CNN
+	1    10700 7000
+	0    1    1    0
+$EndComp
+Wire Wire Line
+	10600 7000 9150 7000
+$Comp
+L power:GND #PWR?
+U 1 1 5FF12FB8
+P 11250 7000
+F 0 "#PWR?" H 11250 6750 50  0001 C CNN
+F 1 "GND" V 11255 6872 50  0000 R CNN
+F 2 "" H 11250 7000 50  0001 C CNN
+F 3 "" H 11250 7000 50  0001 C CNN
+	1    11250 7000
+	0    -1   -1   0
+$EndComp
+Wire Wire Line
+	11250 7000 10800 7000
 $EndSCHEMATC

Commit message: Schematic update
Schematic update - Page 3.
Parts:
- added C?: C, symbol Device:C
- added R?: 10k, symbol Device:R_Small_US
- added R? (x2): 0, symbol Device:R_Small_US
- added R?: 402, symbol Device:R_Small_US
- added TP?: TestPoint, symbol Connector:TestPoint
- added U?: SN74LVC1G14DBV, Package_TO_SOT_SMD:SOT-23-5, symbol 74xGxx:SN74LVC1G14DBV
Connections:
- net GND: now also C?.2, R?.2, R?.2, R?.2, U?.3 (GND)
- net at U?.A29 (RESERVED_A29): now also R?.1
- net at U?.AK12 (DDI0_RCOMP_P): now also R?.2
- net at U?.AK13 (~DDI0_RCOMP): now also R?.1
- net at U?.AM2 (RESERVED_VSS1): now also R?.1
- net at U?.AM3 (RESERVED_VSS0): now also R?.1
- net HDMI_CLK_DN: now reaches U?.AP2 (DDI0_TXN_3)
- net HDMI_CLK_DP: now reaches U?.AP3 (DDI0_TXP_3)
- net HDMI_TX0_DN: now reaches U?.AR1 (DDI0_TXN_2)
- net HDMI_TX0_DP: now reaches U?.AR3 (DDI0_TXP_2)
- net HDMI_TX1_DP: now reaches U?.AT2 (DDI0_TXP_1)
- net HDMI_TX1_DN: now reaches U?.AT3 (DDI0_TXN_1)
- net HDMI_TX2_DN: now reaches U?.AV2 (DDI0_TXN_0)
- net HDMI_TX2_DP: now reaches U?.AV3 (DDI0_TXP_0)
- net at U?.B30 (GPIO_S0_NC12): now also TP?.1
- net HDMI_HPD_B: now reaches U?.D27 (DDI0_HPD)
- net HDMI_HPD_B: now also U?.4
- net DDI1_DDCDAT: now reaches R?.2, U?.P30 (DDI1_DDCDATA)
- new net +1V8: C?.1, U?.5 (VCC)
- new net HDMI_HPD: U?.2
Changed lines of the file:
@@
 Wire Wire Line
 	11250 7000 10800 7000
+$Comp
+L Device:R_Small_US R?
+U 1 1 5FF63478
+P 6100 6400
+F 0 "R?" V 5895 6400 50  0000 C CNN
+F 1 "10k" V 5986 6400 50  0000 C CNN
+F 2 "" H 6100 6400 50  0001 C CNN
+F 3 "~" H 6100 6400 50  0001 C CNN
+	1    6100 6400
+	0    1    1    0
+$EndComp
+Wire Wire Line
+	7100 6400 6200 6400
+$Comp
+L power:GND #PWR?
+U 1 1 5FF6D050
+P 5600 6400
+F 0 "#PWR?" H 5600 6150 50  0001 C CNN
+F 1 "GND" V 5605 6272 50  0000 R CNN
+F 2 "" H 5600 6400 50  0001 C CNN
+F 3 "" H 5600 6400 50  0001 C CNN
+	1    5600 6400
+	0    1    1    0
+$EndComp
+Wire Wire Line
+	6000 6400 5600 6400
+$Comp
+L Connector:TestPoint TP?
+U 1 1 5FF7270B
+P 6200 6700
+F 0 "TP?" V 6395 6772 50  0000 C CNN
+F 1 "TestPoint" V 6304 6772 50  0000 C CNN
+F 2 "" H 6400 6700 50  0001 C CNN
+F 3 "~" H 6400 6700 50  0001 C CNN
+	1    6200 6700
+	0    -1   -1   0
+$EndComp
+Wire Wire Line
+	7100 6700 6200 6700
+$Comp
+L Device:R_Small_US R?
+U 1 1 5FF7C5C2
+P 6100 4100
+F 0 "R?" V 5895 4100 50  0000 C CNN
+F 1 "0" V 5986 4100 50  0000 C CNN
+F 2 "" H 6100 4100 50  0001 C CNN
+F 3 "~" H 6100 4100 50  0001 C CNN
+	1    6100 4100
+	0    1    1    0
+$EndComp
+Wire Wire Line
+	7100 4100 6200 4100
+$Comp
+L power:GND #PWR?
+U 1 1 5FF7C5C9
+P 5600 4100
+F 0 "#PWR?" H 5600 3850 50  0001 C CNN
+F 1 "GND" V 5605 3972 50  0000 R CNN
+F 2 "" H 5600 4100 50  0001 C CNN
+F 3 "" H 5600 4100 50  0001 C CNN
+	1    5600 4100
+	0    1    1    0
+$EndComp
+Wire Wire Line
+	6000 4100 5600 4100
+$Comp
+L power:GND #PWR?
+U 1 1 5FF7F537
+P 5600 4200
+F 0 "#PWR?" H 5600 3950 50  0001 C CNN
+F 1 "GND" V 5605 4072 50  0000 R CNN
+F 2 "" H 5600 4200 50  0001 C CNN
+F 3 "" H 5600 4200 50  0001 C CNN
+	1    5600 4200
+	0    1    1    0
+$EndComp
+Wire Wire Line
+	5600 4200 6250 4200
+Wire Wire Line
+	7100 4200 6450 4200
+$Comp
+L Device:R_Small_US R?
+U 1 1 5FF7F530
+P 6350 4200
+F 0 "R?" V 6145 4200 50  0000 C CNN
+F 1 "0" V 6236 4200 50  0000 C CNN
+F 2 "" H 6350 4200 50  0001 C CNN
+F 3 "~" H 6350 4200 50  0001 C CNN
+	1    6350 4200
+	0    1    1    0
+$EndComp
+$Comp
+L Device:R_Small_US R?
+U 1 1 5FF9866C
+P 6100 3700
+F 0 "R?" V 5895 3700 50  0000 C CNN
+F 1 "402" V 5986 3700 50  0000 C CNN
+F 2 "" H 6100 3700 50  0001 C CNN
+F 3 "~" H 6100 3700 50  0001 C CNN
+	1    6100 3700
+	0    1    1    0
+$EndComp
+Wire Wire Line
+	7100 3700 6200 3700
+Wire Wire Line
+	6000 3700 5750 3700
+Wire Wire Line
+	5750 3700 5750 3800
+Wire Wire Line
+	5750 3800 7100 3800
+Wire Wire Line
+	7100 1850 6300 1850
+Wire Wire Line
+	7100 1950 6300 1950
+Wire Wire Line
+	7100 2050 6300 2050
+Wire Wire Line
+	7100 2150 6300 2150
+Wire Wire Line
+	7100 2250 6300 2250
+Wire Wire Line
+	7100 2350 6300 2350
+Wire Wire Line
+	7100 2450 6300 2450
+Wire Wire Line
+	7100 2550 6300 2550
+Text Label 6300 1850 0    50   ~ 0
+HDMI_TX2_DP
+Text Label 6300 1950 0    50   ~ 0
+HDMI_TX2_DN
+Text Label 6300 2050 0    50   ~ 0
+HDMI_TX1_DP
+Text Label 6300 2150 0    50   ~ 0
+HDMI_TX1_DN
+Text Label 6300 2250 0    50   ~ 0
+HDMI_TX0_DP
+Text Label 6300 2350 0    50   ~ 0
+HDMI_TX0_DN
+Text Label 6300 2450 0    50   ~ 0
+HDMI_CLK_DP
+Text Label 6300 2550 0    50   ~ 0
+HDMI_CLK_DN
+$Comp
+L 74xGxx:SN74LVC1G14DBV U?
+U 1 1 5FFBAA45
+P 3950 2950
+F 0 "U?" H 4294 2996 50  0000 L CNN
+F 1 "SN74LVC1G14DBV" H 4294 2905 50  0000 L CNN
+F 2 "Package_TO_SOT_SMD:SOT-23-5" H 3950 2700 50  0001 C CNN
+F 3 "http://www.ti.com/lit/ds/symlink/sn74lvc1g14.pdf" H 3950 2950 50  0001 C CNN
+	1    3950 2950
+	1    0    0    -1
+$EndComp
+Wire Wire Line
+	4250 2950 7100 2950
+$Comp
+L Device:C C?
+U 1 1 5FFC0CDF
+P 3000 2100
+F 0 "C?" H 3115 2146 50  0000 L CNN
+F 1 "C" H 3115 2055 50  0000 L CNN
+F 2 "" H 3038 1950 50  0001 C CNN
+F 3 "~" H 3000 2100 50  0001 C CNN
+	1    3000 2100
+	1    0    0    -1
+$EndComp
+$Comp
+L power:GND #PWR?
+U 1 1 5FFC4451
+P 3000 2450
+F 0 "#PWR?" H 3000 2200 50  0001 C CNN
+F 1 "GND" H 3005 2277 50  0000 C CNN
+F 2 "" H 3000 2450 50  0001 C CNN
+F 3 "" H 3000 2450 50  0001 C CNN
+	1    3000 2450
+	1    0    0    -1
+$EndComp
+Wire Wire Line
+	3000 2450 3000 2250
+Wire Wire Line
+	3950 2750 3950 1750
+Wire Wire Line
+	3950 1750 3000 1750
+$Comp
+L power:GND #PWR?
+U 1 1 5FFC8905
+P 3950 3300
+F 0 "#PWR?" H 3950 3050 50  0001 C CNN
+F 1 "GND" H 3955 3127 50  0000 C CNN
+F 2 "" H 3950 3300 50  0001 C CNN
+F 3 "" H 3950 3300 50  0001 C CNN
+	1    3950 3300
+	1    0    0    -1
+$EndComp
+Wire Wire Line
+	3950 3300 3950 3150
+Wire Wire Line
+	3750 2950 2300 2950
+Text Label 2300 2950 0    50   ~ 0
+HDMI_HPD
+$Comp
+L power:+1V8 #PWR?
+U 1 1 5FFCEA5F
+P 3000 1350
+F 0 "#PWR?" H 3000 1200 50  0001 C CNN
+F 1 "+1V8" H 3015 1523 50  0000 C CNN
+F 2 "" H 3000 1350 50  0001 C CNN
+F 3 "" H 3000 1350 50  0001 C CNN
+	1    3000 1350
+	1    0    0    -1
+$EndComp
+Wire Wire Line
+	3000 1350 3000 1750
+Connection ~ 3000 1750
+Wire Wire Line
+	3000 1750 3000 1950
+Text Label 5750 2950 0    50   ~ 0
+HDMI_HPD_B
+Text Label 9700 3100 0    50   ~ 0
+DDI1_DDCDAT
 $EndSCHEMATC
